File: PCB/PCB.kicad_pcb (KiCad board)
At the start: 2 copper layers, 4 parts, among them J1 Ultrasonic Sensor, U1 XL1509-3.3, U2 ESP32-C3-DevKitM-1

Commit message: changed pcb cords
Parts:
- moved BT1 41.8 mm to (118.0, 35.0)
- moved J1 41.8 mm to (116.9, 62.0)
Changed lines of the file:
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@@
 	(footprint "Connector_PinHeader_2.54mm:PinHeader_1x04_P2.54mm_Vertical"
 		(layer "F.Cu")
-		(at 134.265 100.035)
+		(at 116.93 62.03)
 		(descr "Through hole straight pin header, 1x04, 2.54mm pitch, single row")
 		(tags "Through hole pin header THT 1x04 2.54mm single row")
@@
 	(footprint "Battery:BatteryHolder_Keystone_2462_2xAA"
 		(layer "F.Cu")
-		(at 135.335 73.005)
+		(at 118 35)
 		(descr "2xAA cell battery holder, Keystone P/N 2462, https://www.keyelco.com/product-pdf.cfm?p=1027")
 		(tags "AA battery cell holder")

Commit message: trial change
...
Parts:
- moved J1 9.15 mm to (115.3, 53.0)
- moved BT1 9.15 mm to (116.3, 26.0)
Changed lines of the file:
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@@
 	(footprint "Connector_PinHeader_2.54mm:PinHeader_1x04_P2.54mm_Vertical"
 		(layer "F.Cu")
-		(at 116.93 62.03)
+		(at 115.265 53.035)
 		(descr "Through hole straight pin header, 1x04, 2.54mm pitch, single row")
 		(tags "Through hole pin header THT 1x04 2.54mm single row")
@@
 	(footprint "Battery:BatteryHolder_Keystone_2462_2xAA"
 		(layer "F.Cu")
-		(at 118 35)
+		(at 116.335 26.005)
 		(descr "2xAA cell battery holder, Keystone P/N 2462, https://www.keyelco.com/product-pdf.cfm?p=1027")
 		(tags "AA battery cell holder")
