File: PCB/PCB.kicad_pcb (KiCad board)
At the start: 2 copper layers, 4 parts, among them J1 Ultrasonic Sensor, U1 XL1509-3.3, U2 ESP32-C3-DevKitM-1

Commit message: Updated the PCB Layout and updated the connections
Parts:
- added BT2: Battery, Battery:BatteryHolder_Keystone_2462_2xAA, F.Cu at (32.5, 70.0)
- added D2: Green, LED_THT:LED_D5.0mm, F.Cu at (45.2, 22.8)
- added D3: Yellow, LED_THT:LED_D5.0mm, F.Cu at (52.7, 22.8)
- added D4: Yellow, LED_THT:LED_D5.0mm, F.Cu at (60.2, 22.8)
- added D5: Red, LED_THT:LED_D5.0mm, F.Cu at (67.6, 22.8)
- added Green1: LED, LED_THT:LED_D5.0mm, F.Cu at (75.1, 22.8)
- added R1: 56k, Resistor_THT:R_Axial_DIN0207_L6.3mm_D2.5mm_P7.62mm_Horizontal, F.Cu at (58.5, 98.4)
- added R2: 47k, Resistor_THT:R_Axial_DIN0207_L6.3mm_D2.5mm_P7.62mm_Horizontal, F.Cu at (69.4, 98.5)
- added U4: Custom_ESP32_S3_Board, Custom:ESP32-S3-DevKitC, F.Cu at (96.6, 36.6)
- J1: value Ultrasonic Sensor -> NiMH CHARGER CIRCUIT
- U1: value XL1509-3.3 -> Buck Converter; footprint Package_SO:SOIC-8_3.9x4.9mm_P1.27mm -> Connector_PinHeader_2.54mm:PinHeader_1x04_P2.54mm_Vertical
- U2: value ESP32-C3-DevKitM-1 -> Ultrasonic Sensor; footprint RF_Module:ESP32-C3-DevKitM-1 -> Connector_PinHeader_2.54mm:PinHeader_1x04_P2.54mm_Vertical
- moved U2 108.4 mm to (126.0, 56.4)
- moved J1 94.2 mm to (21.2, 56.4)
- moved BT1 84.4 mm to (32.5, 35.5)
- moved U1 75.7 mm to (52.2, 98.5), turned to -90 degrees
Connections:
- BT1 pad 2: GND -> 4SPACK-
- J1 pad 1: Net-(J1-Pin_1) -> 4SPACK+
- J1 pad 2: Net-(J1-Pin_2) -> 4SPACK-
- J1 pad 3: Net-(J1-Pin_3) -> /OUT+
- U1 pad 1: Net-(BT1-+) -> Net-(U1-Pin_1)
- U1 pad 2: Net-(U1-OUT) -> /OUT+
- U1 pad 3: unconnected-(U1-FB-Pad3) -> GND
- U1 pad 4: unconnected-(U1-~{EN}-Pad4) -> GND
- U2 pad 1: GND -> +5V
- U2 pad 2: Net-(U1-OUT) -> TRIG
- U2 pad 3: Net-(U1-OUT) -> ECHO
- U2 pad 4: unconnected-(U2-IO2-Pad4) -> GND

Commit message: PCB optimisation
Parts:
- moved R1 65.8 mm to (124.3, 100.2)
- moved R2 65.8 mm to (135.1, 100.3)
- moved U1 26.4 mm to (77.0, 107.7)
- moved U4 26.4 mm to (121.4, 45.8)
- moved BT1 26.4 mm to (57.3, 44.7)
- moved BT2 26.4 mm to (57.3, 79.2)
- moved D2 26.4 mm to (70.0, 32.0)
- moved D3 26.4 mm to (77.5, 32.0)
- moved D4 26.4 mm to (84.9, 32.0)
- moved D5 26.4 mm to (92.4, 32.0)
- moved Green1 26.4 mm to (99.9, 32.0)
- moved J1 26.4 mm to (45.9, 65.6)
- moved U2 26.4 mm to (150.8, 65.7)
Changed lines of the file:
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@@
 	)
 	(setup
+		(stackup
+			(layer "F.SilkS"
+				(type "Top Silk Screen")
+			)
+			(layer "F.Paste"
+				(type "Top Solder Paste")
+			)
+			(layer "F.Mask"
+				(type "Top Solder Mask")
+				(thickness 0.01)
+			)
+			(layer "F.Cu"
+				(type "copper")
+				(thickness 0.035)
+			)
+			(layer "dielectric 1"
+				(type "core")
+				(thickness 1.51)
+				(material "FR4")
+				(epsilon_r 4.5)
+				(loss_tangent 0.02)
+			)
+			(layer "B.Cu"
+				(type "copper")
+				(thickness 0.035)
+			)
+			(layer "B.Mask"
+				(type "Bottom Solder Mask")
+				(thickness 0.01)
+			)
+			(layer "B.Paste"
+				(type "Bottom Solder Paste")
+			)
+			(layer "B.SilkS"
+				(type "Bottom Silk Screen")
+			)
+			(copper_finish "None")
+			(dielectric_constraints no)
+		)
 		(pad_to_mask_clearance 0)
 		(allow_soldermask_bridges_in_footprints no)
@@
 	(footprint "LED_THT:LED_D5.0mm"
 		(layer "F.Cu")
-		(at 67.635 22.755 90)
+		(at 92.41 32 90)
 		(descr "LED, diameter 5.0mm, 2 pins, http://cdn-reichelt.de/documents/datenblatt/A500/LL-504BC2E-009.pdf, generated by kicad-footprint-generator")
 		(tags "LED")
@@
 		)
 		(point
-			(at 67.635 21.485)
+			(at 92.41 30.73)
 			(size 2)
 			(layer "F.Fab")
@@
 	(footprint "Resistor_THT:R_Axial_DIN0207_L6.3mm_D2.5mm_P7.62mm_Horizontal"
 		(layer "F.Cu")
-		(at 58.545 98.44)
+		(at 124.275 100.245)
 		(descr "Resistor, Axial_DIN0207 series, Axial, Horizontal, pin pitch=7.62mm, 0.25W = 1/4W, length*diameter=6.3*2.5mm^2, http://cdn-reichelt.de/documents/datenblatt/B400/1_4W%23YAG.pdf")
 		(tags "Resistor Axial_DIN0207 series Axial Horizontal pin pitch 7.62mm 0.25W = 1/4W length 6.3mm diameter 2.5mm")
@@
 	(footprint "LED_THT:LED_D5.0mm"
 		(layer "F.Cu")
-		(at 60.165 22.755 90)
+		(at 84.94 32 90)
 		(descr "LED, diameter 5.0mm, 2 pins, http://cdn-reichelt.de/documents/datenblatt/A500/LL-504BC2E-009.pdf, generated by kicad-footprint-generator")
 		(tags "LED")
@@
 		)
 		(point
-			(at 60.165 21.485)
+			(at 84.94 30.73)
 			(size 2)
 			(layer "F.Fab")
@@
 	(footprint "Resistor_THT:R_Axial_DIN0207_L6.3mm_D2.5mm_P7.62mm_Horizontal"
 		(layer "F.Cu")
-		(at 69.355 98.49)
+		(at 135.085 100.295)
 		(descr "Resistor, Axial_DIN0207 series, Axial, Horizontal, pin pitch=7.62mm, 0.25W = 1/4W, length*diameter=6.3*2.5mm^2, http://cdn-reichelt.de/documents/datenblatt/B400/1_4W%23YAG.pdf")
 		(tags "Resistor Axial_DIN0207 series Axial Horizontal pin pitch 7.62mm 0.25W = 1/4W length 6.3mm diameter 2.5mm")
@@
 	(footprint "Custom:ESP32-S3-DevKitC"
 		(layer "F.Cu")
-		(at 96.64 36.56)
+		(at 121.415 45.805)
 		(descr "ESP32-S3 development board custom 2x20 pin footprint; antenna end at top")
 		(tags "ESP32-S3 custom 2x20")
@@
 	(footprint "Battery:BatteryHolder_Keystone_2462_2xAA"
 		(layer "F.Cu")
-		(at 32.5 35.5)
+		(at 57.275 44.745)
 		(descr "2xAA cell battery holder, Keystone P/N 2462, https://www.keyelco.com/product-pdf.cfm?p=1027")
 		(tags "AA battery cell holder")
@@
 	(footprint "Connector_PinHeader_2.54mm:PinHeader_1x04_P2.54mm_Vertical"
 		(layer "F.Cu")
-		(at 52.205 98.49 -90)
+		(at 76.98 107.735 -90)
 		(descr "Through hole straight pin header, 1x04, 2.54mm pitch, single row")
 		(tags "Through hole pin header THT 1x04 2.54mm single row")
 		(property "Reference" "U1"
-			(at 0 -2.38 90)
+			(at -7.44 -43.335 90)
 			(layer "F.SilkS")
 			(effects
@@
 	(footprint "LED_THT:LED_D5.0mm"
 		(layer "F.Cu")
-		(at 52.695 22.755 90)
+		(at 77.47 32 90)
 		(descr "LED, diameter 5.0mm, 2 pins, http://cdn-reichelt.de/documents/datenblatt/A500/LL-504BC2E-009.pdf, generated by kicad-footprint-generator")
 		(tags "LED")
@@
 		)
 		(point
-			(at 52.695 21.485)
+			(at 77.47 30.73)
 			(size 2)
 			(layer "F.Fab")
@@
 	(footprint "LED_THT:LED_D5.0mm"
 		(layer "F.Cu")
-		(at 45.225 22.755 90)
+		(at 70 32 90)
 		(descr "LED, diameter 5.0mm, 2 pins, http://cdn-reichelt.de/documents/datenblatt/A500/LL-504BC2E-009.pdf, generated by kicad-footprint-generator")
 		(tags "LED")
@@
 		)
 		(point
-			(at 45.225 21.485)
+			(at 70 30.73)
 			(size 2)
 			(layer "F.Fab")
@@
 	(footprint "Connector_PinHeader_2.54mm:PinHeader_1x04_P2.54mm_Vertical"
 		(layer "F.Cu")
-		(at 126.02 56.40688)
+		(at 150.795 65.65188)
 		(descr "Through hole straight pin header, 1x04, 2.54mm pitch, single row")
 		(tags "Through hole pin header THT 1x04 2.54mm single row")
@@
 	(footprint "Connector_PinHeader_2.54mm:PinHeader_1x04_P2.54mm_Vertical"
 		(layer "F.Cu")
-		(at 21.165 56.37)
+		(at 45.94 65.615)
 		(descr "Through hole straight pin header, 1x04, 2.54mm pitch, single row")
 		(tags "Through hole pin header THT 1x04 2.54mm single row")
@@
 	(footprint "LED_THT:LED_D5.0mm"
 		(layer "F.Cu")
-		(at 75.105 22.755 90)
+		(at 99.88 32 90)
 		(descr "LED, diameter 5.0mm, 2 pins, http://cdn-reichelt.de/documents/datenblatt/A500/LL-504BC2E-009.pdf, generated by kicad-footprint-generator")
 		(tags "LED")
@@
 		)
 		(point
-			(at 75.105 21.485)
+			(at 99.88 30.73)
 			(size 2)
 			(layer "F.Fab")
@@
 	(footprint "Battery:BatteryHolder_Keystone_2462_2xAA"
 		(layer "F.Cu")
-		(at 32.5 69.98)
+		(at 57.275 79.225)
 		(descr "2xAA cell battery holder, Keystone P/N 2462, https://www.keyelco.com/product-pdf.cfm?p=1027")
 		(tags "AA battery cell holder")

Commit message: removed unused component
Parts:
- removed J1: NiMH CHARGER CIRCUIT, Connector_PinHeader_2.54mm:PinHeader_1x04_P2.54mm_Vertical
Connections:
- D2 pad 1: GND -> 4SPACK-
- D3 pad 1: GND -> 4SPACK-
- D4 pad 1: GND -> 4SPACK-
- D5 pad 1: GND -> 4SPACK-
- Green1 pad 1: GND -> 4SPACK-
- R2 pad 1: GND -> 4SPACK-
- U1 pad 2: /OUT+ -> 4SPACK+
- U1 pad 3: GND -> 4SPACK-
- U1 pad 4: GND -> 4SPACK-
- U2 pad 4: GND -> 4SPACK-
- U4 pad 25: GND -> 4SPACK-

Commit message: .
Parts:
- removed Green1: LED, LED_THT:LED_D5.0mm
- added BZ1: Buzzer, Buzzer_Beeper:Buzzer_TDK_PS1240P02BT_D12.2mm_H6.5mm, F.Cu at (178.6, 93.9)
- added D1: Green, LED_THT:LED_D5.0mm, F.Cu at (155.2, 103.5)
- added R3: 330, Resistor_THT:R_Axial_DIN0207_L6.3mm_D2.5mm_P7.62mm_Horizontal, F.Cu at (153.5, 96.9)
- added R4: 330, Resistor_THT:R_Axial_DIN0207_L6.3mm_D2.5mm_P7.62mm_Horizontal, F.Cu at (157.6, 96.9)
- added R5: 330, Resistor_THT:R_Axial_DIN0207_L6.3mm_D2.5mm_P7.62mm_Horizontal, F.Cu at (161.6, 96.9)
- added R6: 330, Resistor_THT:R_Axial_DIN0207_L6.3mm_D2.5mm_P7.62mm_Horizontal, F.Cu at (165.7, 96.9)
- added R7: 330, Resistor_THT:R_Axial_DIN0207_L6.3mm_D2.5mm_P7.62mm_Horizontal, F.Cu at (169.7, 96.9)
- moved D2 117.1 mm to (162.7, 103.5)
- moved D3 117.1 mm to (170.2, 103.5)
- moved D4 117.1 mm to (177.6, 103.5)
- moved D5 117.1 mm to (185.1, 103.5)
Connections:
- D2 pad 2: GPIO38 -> Net-(D2-A)
- D3 pad 2: GPIO37 -> Net-(D3-A)
- D4 pad 2: GPIO36 -> Net-(D4-A)
- D5 pad 2: GPIO35 -> Net-(D5-A)
- U4 pad 3: unconnected-(U4-GPIO4-Pad3) -> BUZZER+

Commit message: trying_traces
Parts:
- removed BT2: Battery, Battery:BatteryHolder_Keystone_2462_2xAA
- moved R1 105.4 mm to (22.2, 74.0)
- moved R2 105.4 mm to (33.0, 74.0)
- moved U1 64.5 mm to (31.0, 62.5)
- moved D1 40.3 mm to (127.6, 74.1)
- moved BZ1 40.3 mm to (151.0, 64.5)
- moved D2 40.3 mm to (135.1, 74.1)
- moved D3 40.3 mm to (142.6, 74.1)
- moved D4 40.3 mm to (150.0, 74.1)
- moved D5 40.3 mm to (157.5, 74.1)
- moved R3 40.3 mm to (125.9, 67.6)
- moved R4 40.3 mm to (129.9, 67.6)
- moved R5 40.3 mm to (134.0, 67.6)
- moved R6 40.3 mm to (138.1, 67.6)
- moved R7 40.3 mm to (142.1, 67.6)
- moved U2 40.2 mm to (127.0, 33.2)
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Connections:
- BT1 pad 1: Net-(BT1-+) -> 4SPACK+
Routing:
- net Net-(U1-Pin_1): track 0.00 -> 76.5 mm
- net 4SPACK+: track 0.00 -> 54.7 mm
- net 4SPACK-: track 0.00 -> 35.3 mm

Commit message: pcb
Parts:
- removed BT1: Battery, Battery:BatteryHolder_Keystone_2462_2xAA
- removed U1: Buck Converter, Connector_PinHeader_2.54mm:PinHeader_1x04_P2.54mm_Vertical
- removed U4: Custom_ESP32_S3_Board, Custom:ESP32-S3-DevKitC
- added H1: MountingHole, MountingHole:MountingHole_2.2mm_M2_DIN965, F.Cu at (122.3, 53.3)
- added H2: MountingHole, MountingHole:MountingHole_2.2mm_M2_DIN965, F.Cu at (122.3, 87.2)
- added H3: MountingHole, MountingHole:MountingHole_2.2mm_M2_DIN965, F.Cu at (211.2, 53.3)
- added H4: MountingHole, MountingHole:MountingHole_2.2mm_M2_DIN965, F.Cu at (211.2, 87.2)
- added J1: motor, Connector_PinHeader_2.54mm:PinHeader_1x03_P2.54mm_Vertical, F.Cu at (192.1, 53.5)
- added J2: out, Connector_PinHeader_2.54mm:PinHeader_1x02_P2.54mm_Vertical, F.Cu at (166.7, 87.5)
- added J3: in, Connector_PinHeader_2.54mm:PinHeader_1x02_P2.54mm_Vertical, F.Cu at (146.2, 87.5)
- added J4: in, Connector_PinHeader_2.54mm:PinHeader_1x02_P2.54mm_Vertical, F.Cu at (121.5, 70.2)
- added U3: Ultrasonic Sensor, Connector_PinHeader_2.54mm:PinHeader_1x04_P2.54mm_Vertical, F.Cu at (184.0, 87.5)
- added U5: ESP32-DEVKITC-32E, ESP32-DEVKITC-32E:MODULE_ESP32-DEVKITC-32E, F.Cu at (189.6, 70.2)
- moved R1 137.2 mm to (159.3, 77.0), turned to 180 degrees
- moved R2 118.7 mm to (151.7, 74.0)
- moved U2 88.2 mm to (196.5, 87.5), turned to 90 degrees
- moved D1 38.0 mm to (159.4, 53.5), turned to -90 degrees
- moved D5 34.8 mm to (129.6, 53.5), turned to -90 degrees
- moved R3 33.6 mm to (159.5, 66.6)
- moved D2 26.7 mm to (152.0, 53.5), turned to -90 degrees
- moved D4 24.4 mm to (137.0, 53.5), turned to -90 degrees
- moved R4 22.1 mm to (152.0, 66.6)
- moved D3 20.8 mm to (144.5, 53.5), turned to -90 degrees
- moved BZ1 14.0 mm to (143.0, 76.0), turned to 180 degrees
- moved R7 12.6 mm to (129.5, 66.6)
- moved R5 10.5 mm to (144.5, 66.6)
- moved R6 1.41 mm to (137.0, 66.6)
Connections:
- net 4SPACK- renamed GND
- R1 pad 2: 4SPACK+ -> +BATT
- U2 pad 1: +5V -> +3.3V
Routing:
- net Net-(U1-Pin_1): track 76.5 -> 0.00 mm
- net 4SPACK+: track 54.7 -> 0.00 mm
- net BUZZER+: track 0.00 -> 44.4 mm
- net GPIO35: track 0.00 -> 43.6 mm
- net +3.3V: track 0.00 -> 39.9 mm
- net GPIO36: track 0.00 -> 38.6 mm
- net GND: track 35.3 -> 0.00 mm
- net GPIO37: track 0.00 -> 33.8 mm
- net ADC: track 0.00 -> 33.3 mm
- net GPIO38: track 0.00 -> 28.7 mm
- net GPIO39: track 0.00 -> 23.8 mm
- net ECHO: track 0.00 -> 6.36 mm
- net TRIG: track 0.00 -> 6.36 mm
- net TRIG1: track 0.00 -> 5.86 mm
- net ECHO1: track 0.00 -> 5.86 mm
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- added copper zone on F.Cu, net +3.3V
- added copper zone on F.Cu, net +BATT
- added copper zone on B.Cu, net GND
Other:
- board outline added: 95 x 40 mm
- board text added: "designed by ~rajeev"
- board text added: "group 1"

Commit message: PC update
Other:
- board text added: "designed by ~rajeev and Ewen"
- board text removed: "designed by ~rajeev"

Commit message: ..
Parts:
- moved U2 74.8 mm to (122.5, 76.5)
- moved J1 69.8 mm to (122.5, 58.5), turned to 0 degrees
- moved U3 61.8 mm to (122.5, 81.0)
- moved J4 1.99 mm to (122.5, 68.5)
Changed lines of the file:
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@@
 	(footprint "Connector_PinHeader_2.54mm:PinHeader_1x04_P2.54mm_Vertical"
 		(layer "F.Cu")
-		(at 184 87.5 90)
+		(at 122.5 81 90)
 		(descr "Through hole straight pin header, 1x04, 2.54mm pitch, single row")
 		(tags "Through hole pin header THT 1x04 2.54mm single row")
@@
 	(footprint "Connector_PinHeader_2.54mm:PinHeader_1x03_P2.54mm_Vertical"
 		(layer "F.Cu")
-		(at 192.08 53.5 -90)
+		(at 122.5 58.46)
 		(descr "Through hole straight pin header, 1x03, 2.54mm pitch, single row")
 		(tags "Through hole pin header THT 1x03 2.54mm single row")
 		(property "Reference" "J1"
-			(at 0 -2.38 90)
+			(at 0 -2.38 0)
 			(layer "F.SilkS")
 			(effects
@@
 		)
 		(property "Value" "motor"
-			(at 0 7.46 90)
+			(at 0 7.46 0)
 			(layer "F.Fab")
 			(effects
@@
 		)
 		(property "Datasheet" ""
-			(at 0 0 90)
+			(at 0 0 0)
 			(layer "F.Fab")
 			(hide yes)
@@
 		)
 		(property "Description" "Generic connector, single row, 01x03, script generated"
-			(at 0 0 90)
+			(at 0 0 0)
 			(layer "F.Fab")
 			(hide yes)
@@
 		(duplicate_pad_numbers_are_jumpers no)
 		(fp_line
-			(start -1.38 6.46)
-			(end 1.38 6.46)
+			(start -1.38 -1.38)
+			(end 0 -1.38)
 			(stroke
 				(width 0.12)
@@
 		)
 		(fp_line
-			(start -1.38 1.27)
-			(end -1.38 6.46)
+			(start -1.38 0)
+			(end -1.38 -1.38)
 			(stroke
 				(width 0.12)
@@
 		(fp_line
 			(start -1.38 1.27)
-			(end 1.38 1.27)
+			(end -1.38 6.46)
 			(stroke
 				(width 0.12)
@@
 		)
 		(fp_line
-			(start 1.38 1.27)
-			(end 1.38 6.46)
+			(start -1.38 1.27)
+			(end 1.38 1.27)
 			(stroke
 				(width 0.12)
@@
 		)
 		(fp_line
-			(start -1.38 0)
-			(end -1.38 -1.38)
+			(start -1.38 6.46)
+			(end 1.38 6.46)
 			(stroke
 				(width 0.12)
@@
 		)
 		(fp_line
-			(start -1.38 -1.38)
-			(end 0 -1.38)
+			(start 1.38 1.27)
+			(end 1.38 6.46)
 			(stroke
 				(width 0.12)
@@
 		)
 		(fp_line
-			(start -1.27 6.35)
-			(end -1.27 -0.635)
+			(start -1.27 -0.635)
+			(end -0.635 -1.27)
 			(stroke
 				(width 0.1)
@@
 		)
 		(fp_line
-			(start 1.27 6.35)
-			(end -1.27 6.35)
+			(start -1.27 6.35)
+			(end -1.27 -0.635)
 			(stroke
 				(width 0.1)
@@
 		)
 		(fp_line
-			(start -1.27 -0.635)
-			(end -0.635 -1.27)
+			(start -0.635 -1.27)
+			(end 1.27 -1.27)
 			(stroke
 				(width 0.1)
@@
 		)
 		(fp_line
-			(start -0.635 -1.27)
-			(end 1.27 -1.27)
+			(start 1.27 -1.27)
+			(end 1.27 6.35)
 			(stroke
 				(width 0.1)
@@
 		)
 		(fp_line
-			(start 1.27 -1.27)
-			(end 1.27 6.35)
+			(start 1.27 6.35)
+			(end -1.27 6.35)
 			(stroke
 				(width 0.1)
@@
 		)
 		(fp_text user "${REFERENCE}"
-			(at 0 2.54 0)
+			(at 0 2.54 90)
 			(layer "F.Fab")
 			(effects
@@
 		)
 		(pad "1" thru_hole rect
-			(at 0 0 270)
+			(at 0 0)
 			(size 1.7 1.7)
 			(drill 1)
@@
 		)
 		(pad "2" thru_hole circle
-			(at 0 2.54 270)
+			(at 0 2.54)
 			(size 1.7 1.7)
 			(drill 1)
@@
 		)
 		(pad "3" thru_hole circle
-			(at 0 5.08 270)
+			(at 0 5.08)
 			(size 1.7 1.7)
 			(drill 1)
@@
 	(footprint "Connector_PinHeader_2.54mm:PinHeader_1x02_P2.54mm_Vertical"
 		(layer "F.Cu")
-		(at 121.5 70.225)
+		(at 122.5 68.5)
 		(descr "Through hole straight pin header, 1x02, 2.54mm pitch, single row")
 		(tags "Through hole pin header THT 1x02 2.54mm single row")
@@
 	(footprint "Connector_PinHeader_2.54mm:PinHeader_1x04_P2.54mm_Vertical"
 		(layer "F.Cu")
-		(at 196.5 87.5 90)
+		(at 122.5 76.5 90)
 		(descr "Through hole straight pin header, 1x04, 2.54mm pitch, single row")
 		(tags "Through hole pin header THT 1x04 2.54mm single row")
