File: PCB/PCB.kicad_pcb (KiCad board)
At the start: 2 copper layers, 95 x 40 mm, 24 parts, among them J1 motor, J2 out, J3 in, J4 in, U2 Ultrasonic Sensor, U3 Ultrasonic Sensor, U5 ESP32-DEVKITC-32E

Commit message: ...
Parts:
- removed J2: out, Connector_PinHeader_2.54mm:PinHeader_1x02_P2.54mm_Vertical
- removed J3, J4: in, Connector_PinHeader_2.54mm:PinHeader_1x02_P2.54mm_Vertical
- added J6: 5V Reg, Connector_PinHeader_2.54mm:PinHeader_1x03_P2.54mm_Vertical, F.Cu at (187.4, 88.0)
- added J8: in, Connector_PinHeader_2.54mm:PinHeader_1x02_P2.54mm_Vertical, F.Cu at (180.0, 88.0)
- moved J1 69.8 mm to (192.0, 53.0), turned to -90 degrees
Connections:
- J1 pad 1: +3.3V -> +5V
- U2 pad 1: +3.3V -> +5V
- U3 pad 1: +3.3V -> +5V
- U5 pad J2_1: +3.3V -> unconnected-(U5-3V3-PadJ2_1)
- U5 pad J2_19: unconnected-(U5-EXT_5V-PadJ2_19) -> +5V
Routing:
- net ECHO: track 6.36 -> 82.9 mm
- net TRIG: track 6.36 -> 81.4 mm
- net ECHO1: track 5.86 -> 69.4 mm
- net TRIG1: track 5.86 -> 67.5 mm
- net +BATT: track 0.00 -> 42.7 mm
- net +3.3V: track 39.9 -> 0.00 mm
- net Net-(D1-A): track 0.00 -> 3.02 mm
- added copper zone on F.Cu, net +5V
- removed copper zone on F.Cu, net +3.3V
- removed copper zone on F.Cu, net +BATT
