File: PCB/PCB.kicad_sch (KiCad schematic)
At the start: 17 parts, among them U1 Buck Converter, U2 Ultrasonic Sensor, U4 Custom_ESP32_S3_Board

Commit message: .
Parts:
- added BZ1: Buzzer, symbol Device:Buzzer
Connections:
- net GND: now also BZ1.2 (-)
- net BUZZER+: now reaches U4.3 (GPIO4)
- net BUZZER+: now also BZ1.1 (+)
Other:
- note added: "Buzzer"

Commit message: .
Parts:
- BZ1: footprint (none) -> Buzzer_Beeper:Buzzer_TDK_PS1240P02BT_D12.2mm_H6.5mm
- R3, R4, R5, R6, R7: footprint (none) -> Resistor_THT:R_Axial_DIN0207_L6.3mm_D2.5mm_P7.62mm_Horizontal
Changed lines of the file:
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@@
 			)
 		)
-		(property "Footprint" ""
+		(property "Footprint" "Buzzer_Beeper:Buzzer_TDK_PS1240P02BT_D12.2mm_H6.5mm"
 			(at 191.135 68.58 90)
 			(hide yes)
@@
 			)
 		)
-		(property "Footprint" ""
+		(property "Footprint" "Resistor_THT:R_Axial_DIN0207_L6.3mm_D2.5mm_P7.62mm_Horizontal"
 			(at 124.46 98.298 90)
 			(hide yes)
@@
 			)
 		)
-		(property "Footprint" ""
+		(property "Footprint" "Resistor_THT:R_Axial_DIN0207_L6.3mm_D2.5mm_P7.62mm_Horizontal"
 			(at 124.46 142.748 90)
 			(hide yes)
@@
 			)
 		)
-		(property "Footprint" ""
+		(property "Footprint" "Resistor_THT:R_Axial_DIN0207_L6.3mm_D2.5mm_P7.62mm_Horizontal"
 			(at 124.46 131.318 90)
 			(hide yes)
@@
 			)
 		)
-		(property "Footprint" ""
+		(property "Footprint" "Resistor_THT:R_Axial_DIN0207_L6.3mm_D2.5mm_P7.62mm_Horizontal"
 			(at 124.46 108.458 90)
 			(hide yes)
@@
 			)
 		)
-		(property "Footprint" ""
+		(property "Footprint" "Resistor_THT:R_Axial_DIN0207_L6.3mm_D2.5mm_P7.62mm_Horizontal"
 			(at 124.46 119.888 90)
 			(hide yes)

Commit message: trying_traces
Parts:
- removed BT1: Battery, Battery:BatteryHolder_Keystone_2462_2xAA, symbol Device:Battery
- renumbered BT2 to BT1
Connections:
- net GND: now also BT1.2 (-)
Changed lines of the file:
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@@
 	(rectangle
 		(start 68.58 92.71)
-		(end 97.79 109.22)
+		(end 85.09 109.22)
 		(stroke
 			(width 0)
@@
 	(text "4S Battery\n"
 		(exclude_from_sim no)
-		(at 83.312 110.744 0)
+		(at 77.47 111.252 0)
 		(effects
 			(font
@@
 	(wire
 		(pts
+			(xy 80.01 90.17) (xy 80.01 106.68)
+		)
+		(stroke
+			(width 0)
+			(type default)
+		)
+	)
+	(wire
+		(pts
 			(xy 137.16 129.54) (xy 143.51 129.54)
 		)
@@
 	(wire
 		(pts
-			(xy 80.01 93.98) (xy 80.01 106.68)
-		)
-		(stroke
-			(width 0)
-			(type default)
-		)
-	)
-	(wire
-		(pts
 			(xy 120.65 140.97) (xy 118.11 140.97)
 		)
@@
 	(wire
 		(pts
-			(xy 86.36 106.68) (xy 92.71 106.68)
-		)
-		(stroke
-			(width 0)
-			(type default)
-		)
-	)
-	(wire
-		(pts
 			(xy 128.27 106.68) (xy 129.54 106.68)
 		)
@@
 	(wire
 		(pts
-			(xy 86.36 93.98) (xy 86.36 96.52)
-		)
-		(stroke
-			(width 0)
-			(type default)
-		)
-	)
-	(wire
-		(pts
 			(xy 128.27 96.52) (xy 129.54 96.52)
 		)
@@
 	(wire
 		(pts
-			(xy 86.36 93.98) (xy 80.01 93.98)
-		)
-		(stroke
-			(width 0)
-			(type default)
-		)
-	)
-	(wire
-		(pts
 			(xy 201.93 109.22) (xy 203.2 109.22)
 		)
@@
 	(wire
 		(pts
+			(xy 80.01 90.17) (xy 83.82 90.17)
+		)
+		(stroke
+			(width 0)
+			(type default)
+		)
+	)
+	(wire
+		(pts
 			(xy 77.47 128.27) (xy 76.2 128.27)
 		)
@@
 	(wire
 		(pts
-			(xy 92.71 90.17) (xy 92.71 106.68)
-		)
-		(stroke
-			(width 0)
-			(type default)
-		)
-	)
-	(wire
-		(pts
-			(xy 72.39 90.17) (xy 72.39 96.52)
+			(xy 72.39 87.63) (xy 72.39 96.52)
 		)
 		(stroke
@@
 	(global_label "4SPACK-"
 		(shape input)
-		(at 92.71 90.17 0)
+		(at 83.82 90.17 0)
 		(fields_autoplaced yes)
 		(effects
@@
 		)
 		(property "Intersheetrefs" "${INTERSHEET_REFS}"
-			(at 104.5852 90.17 0)
+			(at 95.6952 90.17 0)
 			(hide yes)
 			(show_name no)
@@
 	(global_label "4SPACK+"
 		(shape input)
-		(at 72.39 90.17 0)
+		(at 72.39 87.63 0)
 		(fields_autoplaced yes)
 		(effects
@@
 		)
 		(property "Intersheetrefs" "${INTERSHEET_REFS}"
-			(at 84.2652 90.17 0)
+			(at 84.2652 87.63 0)
 			(hide yes)
 			(show_name no)
@@
 		(dnp no)
 		(fields_autoplaced yes)
-		(property "Reference" "BT2"
+		(property "Reference" "BT1"
 			(at 76.2 99.7584 0)
 			(show_name no)
@@
 			(project "PCB"
 				(path "/ab40fc32-b885-4754-9572-45a5defa6a02"
-					(reference "BT2")
+					(reference "BT1")
 					(unit 1)
 				)
@@
 					(unit 1)
 				)
-			)
-		)
-	)
-	(symbol
-		(lib_id "Device:Battery")
-		(at 86.36 101.6 0)
-		(unit 1)
-		(body_style 1)
-		(exclude_from_sim no)
-		(in_bom yes)
-		(on_board yes)
-		(in_pos_files yes)
-		(dnp no)
-		(fields_autoplaced yes)
-		(property "Reference" "BT1"
-			(at 90.17 99.7584 0)
-			(show_name no)
-			(do_not_autoplace no)
-			(effects
-				(font
-					(size 1.27 1.27)
-				)
-				(justify left)
-			)
-		)
-		(property "Value" "Battery"
-			(at 90.17 102.2984 0)
-			(show_name no)
-			(do_not_autoplace no)
-			(effects
-				(font
-					(size 1.27 1.27)
-				)
-				(justify left)
-			)
-		)
-		(property "Footprint" "Battery:BatteryHolder_Keystone_2462_2xAA"
-			(at 86.36 100.076 90)
-			(hide yes)
-			(show_name no)
-			(do_not_autoplace no)
-			(effects
-				(font
-					(size 1.27 1.27)
-				)
-			)
-		)
-		(property "Datasheet" ""
-			(at 86.36 100.076 90)
-			(hide yes)
-			(show_name no)
-			(do_not_autoplace no)
-			(effects
-				(font
-					(size 1.27 1.27)
-				)
-			)
-		)
-		(property "Description" "Multiple-cell battery"
-			(at 86.36 101.6 0)
-			(hide yes)
-			(show_name no)
-			(do_not_autoplace no)
-			(effects
-				(font
-					(size 1.27 1.27)
-				)
-			)
-		)
-		(pin "1"
-		)
-		(pin "2"
-		)
-		(instances
-			(project "PCB"
-				(path "/ab40fc32-b885-4754-9572-45a5defa6a02"
-					(reference "BT1")
-					(unit 1)
-				)

Commit message: pcb
Parts:
- removed BT1: Battery, Battery:BatteryHolder_Keystone_2462_2xAA, symbol Device:Battery
- added H1, H2, H3, H4: MountingHole, MountingHole:MountingHole_2.2mm_M2_DIN965, symbol Mechanical:MountingHole
- added J1: motor, Connector_PinHeader_2.54mm:PinHeader_1x03_P2.54mm_Vertical, symbol Connector:Conn_01x03_Socket
- added J2: out, Connector_PinHeader_2.54mm:PinHeader_1x02_P2.54mm_Vertical, symbol Connector:Conn_01x02_Socket
- added J3, J4: in, Connector_PinHeader_2.54mm:PinHeader_1x02_P2.54mm_Vertical, symbol Connector:Conn_01x02_Socket
- added U3: Ultrasonic Sensor, Connector_PinHeader_2.54mm:PinHeader_1x04_P2.54mm_Vertical, symbol Connector_Generic:Conn_01x04
- added U5: ESP32-DEVKITC-32E, ESP32-DEVKITC-32E:MODULE_ESP32-DEVKITC-32E, symbol ESP32-DEVKITC-32E:ESP32-DEVKITC-32E
Connections:
- net +5V is gone; now on net +3.3V: U2.1 (Pin_1)
- net ADC: now also U5.J2_9 (IO25)
- net BUZZER+: now also U5.J2_8 (IO33)
- net ECHO: now also U5.J2_13 (IO12)
- net GND: now also J1.3 (Pin_3), J2.2 (Pin_2), J3.2 (Pin_2), J4.2 (Pin_2), U3.4 (Pin_4), U5.J3_1 (GND_J3_1), U5.J3_7 (GND_J3_7)
- net GPIO35: now also U5.J3_2 (IO23)
- net GPIO36: now also U5.J3_3 (IO22)
- net GPIO37: now also U5.J3_4 (TXD0)
- net GPIO38: now also U5.J3_5 (RXD0)
- net GPIO39: now also U5.J3_6 (IO21)
- net TRIG: now also U5.J2_12 (IO14)
- net +3.3V: now reaches U1.1 (Pin_1), U4.1 (3V3)
- net +3.3V: now also J1.1 (Pin_1), J2.1 (Pin_1), U3.1 (Pin_1), U5.J2_1 (3V3)
- net ECHO1: now reaches U4.10 (GPIO18)
- net ECHO1: now also U3.3 (Pin_3), U5.J2_11 (IO27)
- net TRIG1: now reaches U4.9 (GPIO17)
- net TRIG1: now also U3.2 (Pin_2), U5.J2_10 (IO26)
- net 4SPACK+ renamed +BATT
- net +BATT: now also J3.1 (Pin_1), J4.1 (Pin_1)
- new net SIG: J1.2 (Pin_2), U5.J3_10 (IO5)
Other:
- note added: "buck conveter"
- note added: "motor"
- note added: "sensor"
- moved on the sheet: BZ1, D1, D2, D3, D4, D5, R1, R2, R3, R4, R5, R6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

Commit message: ..
Parts:
- removed J2: out, Connector_PinHeader_2.54mm:PinHeader_1x02_P2.54mm_Vertical, symbol Connector:Conn_01x02_Socket
- removed J3, J4: in, Connector_PinHeader_2.54mm:PinHeader_1x02_P2.54mm_Vertical, symbol Connector:Conn_01x02_Socket
- removed U1: Buck Converter, Connector_PinHeader_2.54mm:PinHeader_1x04_P2.54mm_Vertical, symbol Connector_Generic:Conn_01x04
- added J6: 5V Reg, Connector_PinHeader_2.54mm:PinHeader_1x03_P2.54mm_Vertical, symbol Connector:Conn_01x03_Socket
- added J8: in, Connector_PinHeader_2.54mm:PinHeader_1x02_P2.54mm_Vertical, symbol Connector:Conn_01x02_Socket
Connections:
- net +BATT: now also J6.1 (Pin_1), J8.1 (Pin_1)
- net GND: now also J6.2 (Pin_2), J8.2 (Pin_2)
- new net +5V: J6.3 (Pin_3)
Other:
- note added: "5V Regulator (S9V11F5)"
- note added: "Battery Input"
- note removed: "buck conveter"
- moved on the sheet: U5

Commit message: ...
Connections:
- net +3.3V: no longer J1.1 (Pin_1), U2.1 (Pin_1), U3.1 (Pin_1), U5.J2_1 (3V3)
- net +5V: now also J1.1 (Pin_1), U2.1 (Pin_1), U3.1 (Pin_1), U5.J2_19 (EXT_5V)
Other:
- moved on the sheet: J8
